File: hardware/kicad/R3_PowerBox/R3_power_preiso_buck1.kicad_sch (KiCad schematic)
At the start: 19 parts, among them U2 TPS54302DDCR

Commit message: Rev.A review fixes: local charger power-stage reroute checkpoint
Parts:
- C23, C24: value 22uF/10V -> 22uF/25V GRM32ER71E226KE15L; footprint Capacitor_SMD:C_0805_2012Metric -> Capacitor_SMD:C_1210_3225Metric
Changed lines of the file:
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@@
     (instances
       (project "SKiDL-Generated"
-        (path "/7d40ec76-f97b-4a90-b5ea-ddf1628062b5/10a79bc1-5fff-5d5a-9873-ba1a5dc253c9"
+        (path "/2b0a7443-ac4c-4207-8273-267cee2a0847/10a79bc1-5fff-5d5a-9873-ba1a5dc253c9"
           (reference "U2")
           (unit 1)))))
@@
     (instances
       (project "SKiDL-Generated"
-        (path "/7d40ec76-f97b-4a90-b5ea-ddf1628062b5/10a79bc1-5fff-5d5a-9873-ba1a5dc253c9"
+        (path "/2b0a7443-ac4c-4207-8273-267cee2a0847/10a79bc1-5fff-5d5a-9873-ba1a5dc253c9"
           (reference "L2")
           (unit 1)))))
@@
     (instances
       (project "SKiDL-Generated"
-        (path "/7d40ec76-f97b-4a90-b5ea-ddf1628062b5/10a79bc1-5fff-5d5a-9873-ba1a5dc253c9"
+        (path "/2b0a7443-ac4c-4207-8273-267cee2a0847/10a79bc1-5fff-5d5a-9873-ba1a5dc253c9"
           (reference "C20")
           (unit 1)))))
@@
     (instances
       (project "SKiDL-Generated"
-        (path "/7d40ec76-f97b-4a90-b5ea-ddf1628062b5/10a79bc1-5fff-5d5a-9873-ba1a5dc253c9"
+        (path "/2b0a7443-ac4c-4207-8273-267cee2a0847/10a79bc1-5fff-5d5a-9873-ba1a5dc253c9"
           (reference "C21")
           (unit 1)))))
@@
     (instances
       (project "SKiDL-Generated"
-        (path "/7d40ec76-f97b-4a90-b5ea-ddf1628062b5/10a79bc1-5fff-5d5a-9873-ba1a5dc253c9"
+        (path "/2b0a7443-ac4c-4207-8273-267cee2a0847/10a79bc1-5fff-5d5a-9873-ba1a5dc253c9"
           (reference "C22")
           (unit 1)))))
@@
           (size 0.9 0.9))
         (justify left)))
-    (property "Value" "22uF/10V"
+    (property "Value" "22uF/25V GRM32ER71E226KE15L"
       (at 125 67.54 0)
       (effects
@@
           (size 0.9 0.9))
         (justify left)))
-    (property "Footprint" "Capacitor_SMD:C_0805_2012Metric"
+    (property "Footprint" "Capacitor_SMD:C_1210_3225Metric"
       (at 125 65 0)
       (effects
@@
     (instances
       (project "SKiDL-Generated"
-        (path "/7d40ec76-f97b-4a90-b5ea-ddf1628062b5/10a79bc1-5fff-5d5a-9873-ba1a5dc253c9"
+        (path "/2b0a7443-ac4c-4207-8273-267cee2a0847/10a79bc1-5fff-5d5a-9873-ba1a5dc253c9"
           (reference "C23")
           (unit 1)))))
@@
           (size 0.9 0.9))
         (justify left)))
-    (property "Value" "22uF/10V"
+    (property "Value" "22uF/25V GRM32ER71E226KE15L"
       (at 155 67.54 0)
       (effects
@@
           (size 0.9 0.9))
         (justify left)))
-    (property "Footprint" "Capacitor_SMD:C_0805_2012Metric"
+    (property "Footprint" "Capacitor_SMD:C_1210_3225Metric"
       (at 155 65 0)
       (effects
@@
     (instances
       (project "SKiDL-Generated"
-        (path "/7d40ec76-f97b-4a90-b5ea-ddf1628062b5/10a79bc1-5fff-5d5a-9873-ba1a5dc253c9"
+        (path "/2b0a7443-ac4c-4207-8273-267cee2a0847/10a79bc1-5fff-5d5a-9873-ba1a5dc253c9"
           (reference "C24")
           (unit 1)))))
@@
     (instances
       (project "SKiDL-Generated"
-        (path "/7d40ec76-f97b-4a90-b5ea-ddf1628062b5/10a79bc1-5fff-5d5a-9873-ba1a5dc253c9"
+        (path "/2b0a7443-ac4c-4207-8273-267cee2a0847/10a79bc1-5fff-5d5a-9873-ba1a5dc253c9"
           (reference "R21")
           (unit 1)))))
@@
     (instances
       (project "SKiDL-Generated"
-        (path "/7d40ec76-f97b-4a90-b5ea-ddf1628062b5/10a79bc1-5fff-5d5a-9873-ba1a5dc253c9"
+        (path "/2b0a7443-ac4c-4207-8273-267cee2a0847/10a79bc1-5fff-5d5a-9873-ba1a5dc253c9"
           (reference "R22")
           (unit 1)))))
@@
     (instances
       (project "SKiDL-Generated"
-        (path "/7d40ec76-f97b-4a90-b5ea-ddf1628062b5/10a79bc1-5fff-5d5a-9873-ba1a5dc253c9"
+        (path "/2b0a7443-ac4c-4207-8273-267cee2a0847/10a79bc1-5fff-5d5a-9873-ba1a5dc253c9"
           (reference "C25")
           (unit 1)))))
@@
     (instances
       (project "SKiDL-Generated"
-        (path "/7d40ec76-f97b-4a90-b5ea-ddf1628062b5/10a79bc1-5fff-5d5a-9873-ba1a5dc253c9"
+        (path "/2b0a7443-ac4c-4207-8273-267cee2a0847/10a79bc1-5fff-5d5a-9873-ba1a5dc253c9"
           (reference "FB6")
           (unit 1)))))
@@
     (instances
       (project "SKiDL-Generated"
-        (path "/7d40ec76-f97b-4a90-b5ea-ddf1628062b5/10a79bc1-5fff-5d5a-9873-ba1a5dc253c9"
+        (path "/2b0a7443-ac4c-4207-8273-267cee2a0847/10a79bc1-5fff-5d5a-9873-ba1a5dc253c9"
           (reference "C26")
           (unit 1)))))
@@
     (instances
       (project "SKiDL-Generated"
-        (path "/7d40ec76-f97b-4a90-b5ea-ddf1628062b5/10a79bc1-5fff-5d5a-9873-ba1a5dc253c9"
+        (path "/2b0a7443-ac4c-4207-8273-267cee2a0847/10a79bc1-5fff-5d5a-9873-ba1a5dc253c9"
           (reference "C27")
           (unit 1)))))
@@
     (instances
       (project "SKiDL-Generated"
-        (path "/7d40ec76-f97b-4a90-b5ea-ddf1628062b5/10a79bc1-5fff-5d5a-9873-ba1a5dc253c9"
+        (path "/2b0a7443-ac4c-4207-8273-267cee2a0847/10a79bc1-5fff-5d5a-9873-ba1a5dc253c9"
           (reference "FB7")
           (unit 1)))))
@@
     (instances
       (project "SKiDL-Generated"
-        (path "/7d40ec76-f97b-4a90-b5ea-ddf1628062b5/10a79bc1-5fff-5d5a-9873-ba1a5dc253c9"
+        (path "/2b0a7443-ac4c-4207-8273-267cee2a0847/10a79bc1-5fff-5d5a-9873-ba1a5dc253c9"
           (reference "C28")
           (unit 1)))))
@@
     (instances
       (project "SKiDL-Generated"
-        (path "/7d40ec76-f97b-4a90-b5ea-ddf1628062b5/10a79bc1-5fff-5d5a-9873-ba1a5dc253c9"
+        (path "/2b0a7443-ac4c-4207-8273-267cee2a0847/10a79bc1-5fff-5d5a-9873-ba1a5dc253c9"
           (reference "C29")
           (unit 1)))))
@@
     (instances
       (project "SKiDL-Generated"
-        (path "/7d40ec76-f97b-4a90-b5ea-ddf1628062b5/10a79bc1-5fff-5d5a-9873-ba1a5dc253c9"
+        (path "/2b0a7443-ac4c-4207-8273-267cee2a0847/10a79bc1-5fff-5d5a-9873-ba1a5dc253c9"
           (reference "TP5")
           (unit 1)))))
@@
     (instances
       (project "SKiDL-Generated"
-        (path "/7d40ec76-f97b-4a90-b5ea-ddf1628062b5/10a79bc1-5fff-5d5a-9873-ba1a5dc253c9"
+        (path "/2b0a7443-ac4c-4207-8273-267cee2a0847/10a79bc1-5fff-5d5a-9873-ba1a5dc253c9"
           (reference "TP6")
           (unit 1)))))
@@
     (instances
       (project "SKiDL-Generated"
-        (path "/7d40ec76-f97b-4a90-b5ea-ddf1628062b5/10a79bc1-5fff-5d5a-9873-ba1a5dc253c9"
+        (path "/2b0a7443-ac4c-4207-8273-267cee2a0847/10a79bc1-5fff-5d5a-9873-ba1a5dc253c9"
           (reference "TP16")
           (unit 1)))))
